Commit message: Added D435 gazebo Plugin (two xacro files and command in mir_200_vi.urdf.xacro). Published Topics, namespace and tf_prefix are still not correct. But at least gazebo and rviz open and publish sth.

File: MiR200-with-UR5/mir_ur5_description/urdf/include/mir_200.gazebo.xacro (robot description, xacro)
@@ -58,5 +58,5 @@
   </xacro:macro>
     <!-- camera -->
-    <gazebo reference="robot1_tf/camera_link">
+    <!--gazebo reference="robot1_tf/camera_link">
       <sensor type="depth" name="camera">
         <plugin name="kinect_camera_controller" filename="libgazebo_ros_openni_kinect.so">
@@ -79,4 +79,4 @@
         </plugin>
       </sensor>
-    </gazebo>
+    </gazebo-->
 </robot>

File: MiR200-with-UR5/mir_ur5_description/urdf/mir_200_v1.urdf.xacro (robot description, xacro)
@@ -9,4 +9,5 @@
   <xacro:include filename="$(find mir_ur5_description)/urdf/include/mir_200.transmission.xacro" />
   <xacro:include filename="$(find mir_ur5_description)/urdf/include/sick_s300.urdf.xacro" />
+  <xacro:include filename="$(find mir_ur5_description)/urdf/include/_d435.urdf.xacro"/>
   <xacro:property name="deg_to_rad" value="0.017453293" />
   <xacro:property name="mir_200_base_mass" value="58.0" />
@@ -219,5 +220,6 @@
     <p3d_base_controller prefix="${prefix}" />
     <!-- Camera -->
-    <link name="${prefix}camera_link">
+    <!-- (origin of camera_joint is position of realsense) -->
+     <!--link name="${prefix}camera_link">
       <collision>
         <origin xyz="0 0 0" rpy="0 0 0"/>
@@ -240,13 +242,9 @@
     <joint name="${prefix}camera_joint" type="fixed">
       <axis xyz="0 1 0" />
-      <origin xyz="0.42 0 0.27" rpy="0 0.2 0"/> <!--set the position of the realsense-->
+      <origin xyz="0.42 0 0.27" rpy="0 0.2 0"/>
       <parent link="${prefix}base_link"/>
       <child link="${prefix}camera_link"/>
     </joint>
-    <!-- generate an optical frame http://www.ros.org/reps/rep-0103.html#suffix-frames
-        so that ros and opencv can operate on the camera frame correctly -->
     <joint name="${prefix}camera_optical_joint" type="fixed">
-      <!-- these values have to be these values otherwise the gazebo camera image
-          won't be aligned properly with the frame it is supposedly originating from -->
       <origin xyz="0 0 0" rpy="-1.5708 0 -1.5708"/>
       <parent link="${prefix}camera_link"/>
@@ -254,5 +252,12 @@
     </joint>
     <link name="${prefix}camera_link_optical">
-    </link>
+    </link> -->
+    <!-- generate an optical frame http://www.ros.org/reps/rep-0103.html#suffix-frames
+        so that ros and opencv can operate on the camera frame correctly -->
+    <!-- these values have to be these values otherwise the gazebo camera image
+        won't be aligned properly with the frame it is supposedly originating from -->
+    <xacro:sensor_d435 parent="${prefix}base_link">
+      <origin xyz="0.42 0 0.27" rpy="0 0.2 0"/>
+    </xacro:sensor_d435>
   </xacro:macro>
 </robot>
