Commit message: Added gazebo IntelRealsense Plugin _d435 with correct tf tree names (with prefix). But Published Topics still not correct!

File: MiR200-with-UR5/mir_ur5_description/urdf/include/_d435.urdf.xacro (robot description, xacro)
@@ -9,5 +9,5 @@
   <!--File includes-->
   <xacro:include filename="$(find mir_ur5_description)/urdf/include/_d435.gazebo.xacro"/>
-  <xacro:macro name="sensor_d435" params="name:=camera topics_ns:=camera parent *origin">
+  <xacro:macro name="sensor_d435" params="name:=camera topics_ns:=camera parent tf_prefix *origin">
     <xacro:property name="M_PI" value="3.1415926535897931" />
     <!-- The following values are approximate, and the camera node
@@ -32,16 +32,16 @@
     </material>
     <!-- camera body, with origin at bottom screw mount -->
-    <joint name="${name}_joint" type="fixed">
+    <joint name="${tf_prefix}${name}_joint" type="fixed">
       <xacro:insert_block name="origin" />
       <parent link="${parent}"/>
-      <child link="${name}_bottom_screw_frame" />
+      <child link="${tf_prefix}${name}_bottom_screw_frame" />
     </joint>
-    <link name="${name}_bottom_screw_frame"/>
-    <joint name="${name}_link_joint" type="fixed">
+    <link name="${tf_prefix}${name}_bottom_screw_frame"/>
+    <joint name="${tf_prefix}${name}_link_joint" type="fixed">
       <origin xyz="0 ${d435_cam_depth_py} ${d435_cam_depth_pz}" rpy="0 0 0"/>
-      <parent link="${name}_bottom_screw_frame"/>
-      <child link="${name}_link" />
+      <parent link="${tf_prefix}${name}_bottom_screw_frame"/>
+      <child link="${tf_prefix}${name}_link" />
     </joint>
-    <link name="${name}_link">
+    <link name="${tf_prefix}${name}_link">
       <visual>
       <origin xyz="${d435_cam_mount_from_center_offset} ${-d435_cam_depth_py} 0" rpy="${M_PI/2} 0 ${M_PI/2}"/>
@@ -67,57 +67,57 @@
     </link>
     <!-- camera depth joints and links -->
-    <joint name="${name}_depth_joint" type="fixed">
+    <joint name="${tf_prefix}${name}_depth_joint" type="fixed">
       <origin xyz="0 0 0" rpy="0 0 0"/>
-      <parent link="${name}_link"/>
-      <child link="${name}_depth_frame" />
+      <parent link="${tf_prefix}${name}_link"/>
+      <child link="${tf_prefix}${name}_depth_frame" />
     </joint>
-    <link name="${name}_depth_frame"/>
-    <joint name="${name}_depth_optical_joint" type="fixed">
+    <link name="${tf_prefix}${name}_depth_frame"/>
+    <joint name="${tf_prefix}${name}_depth_optical_joint" type="fixed">
       <origin xyz="0 0 0" rpy="${-M_PI/2} 0 ${-M_PI/2}" />
-      <parent link="${name}_depth_frame" />
-      <child link="${name}_depth_optical_frame" />
+      <parent link="${tf_prefix}${name}_depth_frame" />
+      <child link="${tf_prefix}${name}_depth_optical_frame" />
     </joint>
-    <link name="${name}_depth_optical_frame"/>
+    <link name="${tf_prefix}${name}_depth_optical_frame"/>
     <!-- camera left IR joints and links -->
-    <joint name="${name}_left_ir_joint" type="fixed">
+    <joint name="${tf_prefix}${name}_left_ir_joint" type="fixed">
       <origin xyz="0 ${d435_cam_depth_to_left_ir_offset} 0" rpy="0 0 0" />
-      <parent link="${name}_depth_frame" />
-      <child link="${name}_left_ir_frame" />
+      <parent link="${tf_prefix}${name}_depth_frame" />
+      <child link="${tf_prefix}${name}_left_ir_frame" />
     </joint>
-    <link name="${name}_left_ir_frame"/>
-    <joint name="${name}_left_ir_optical_joint" type="fixed">
+    <link name="${tf_prefix}${name}_left_ir_frame"/>
+    <joint name="${tf_prefix}${name}_left_ir_optical_joint" type="fixed">
       <origin xyz="0 0 0" rpy="${-M_PI/2} 0 ${-M_PI/2}" />
-      <parent link="${name}_left_ir_frame" />
-      <child link="${name}_left_ir_optical_frame" />
+      <parent link="${tf_prefix}${name}_left_ir_frame" />
+      <child link="${tf_prefix}${name}_left_ir_optical_frame" />
     </joint>
-    <link name="${name}_left_ir_optical_frame"/>
+    <link name="${tf_prefix}${name}_left_ir_optical_frame"/>
     <!-- camera right IR joints and links -->
-    <joint name="${name}_right_ir_joint" type="fixed">
+    <joint name="${tf_prefix}${name}_right_ir_joint" type="fixed">
       <origin xyz="0 ${d435_cam_depth_to_right_ir_offset} 0" rpy="0 0 0" />
-      <parent link="${name}_depth_frame" />
-      <child link="${name}_right_ir_frame" />
+      <parent link="${tf_prefix}${name}_depth_frame" />
+      <child link="${tf_prefix}${name}_right_ir_frame" />
     </joint>
-    <link name="${name}_right_ir_frame"/>
-    <joint name="${name}_right_ir_optical_joint" type="fixed">
+    <link name="${tf_prefix}${name}_right_ir_frame"/>
+    <joint name="${tf_prefix}${name}_right_ir_optical_joint" type="fixed">
       <origin xyz="0 0 0" rpy="${-M_PI/2} 0 ${-M_PI/2}" />
-      <parent link="${name}_right_ir_frame" />
-      <child link="${name}_right_ir_optical_frame" />
+      <parent link="${tf_prefix}${name}_right_ir_frame" />
+      <child link="${tf_prefix}${name}_right_ir_optical_frame" />
     </joint>
-    <link name="${name}_right_ir_optical_frame"/>
+    <link name="${tf_prefix}${name}_right_ir_optical_frame"/>
     <!-- camera color joints and links -->
-    <joint name="${name}_color_joint" type="fixed">
+    <joint name="${tf_prefix}${name}_color_joint" type="fixed">
       <origin xyz="0 ${d435_cam_depth_to_color_offset} 0" rpy="0 0 0" />
-      <parent link="${name}_depth_frame" />
-      <child link="${name}_color_frame" />
+      <parent link="${tf_prefix}${name}_depth_frame" />
+      <child link="${tf_prefix}${name}_color_frame" />
     </joint>
-    <link name="${name}_color_frame"/>
-    <joint name="${name}_color_optical_joint" type="fixed">
+    <link name="${tf_prefix}${name}_color_frame"/>
+    <joint name="${tf_prefix}${name}_color_optical_joint" type="fixed">
       <origin xyz="0 0 0" rpy="${-M_PI/2} 0 ${-M_PI/2}" />
-      <parent link="${name}_color_frame" />
-      <child link="${name}_color_optical_frame" />
+      <parent link="${tf_prefix}${name}_color_frame" />
+      <child link="${tf_prefix}${name}_color_optical_frame" />
     </joint>
-    <link name="${name}_color_optical_frame"/>
+    <link name="${tf_prefix}${name}_color_optical_frame"/>
     <!-- Realsense Gazebo Plugin -->
-    <xacro:gazebo_d435 camera_name="${name}" reference_link="${name}_link" topics_ns="${topics_ns}" depth_optical_frame="${name}_depth_optical_frame" color_optical_frame="${name}_color_optical_frame" infrared1_optical_frame="${name}_left_ir_optical_frame" infrared2_optical_frame="${name}_right_ir_optical_frame"/>
+    <xacro:gazebo_d435 camera_name="${name}" reference_link="${tf_prefix}${name}_link" topics_ns="${topics_ns}" depth_optical_frame="${tf_prefix}${name}_depth_optical_frame" color_optical_frame="${tf_prefix}${name}_color_optical_frame" infrared1_optical_frame="${tf_prefix}${name}_left_ir_optical_frame" infrared2_optical_frame="${tf_prefix}${name}_right_ir_optical_frame"/>
   </xacro:macro>
 </robot>

File: MiR200-with-UR5/mir_ur5_description/urdf/mir_200_v1.urdf.xacro (robot description, xacro)
@@ -257,5 +257,5 @@
     <!-- these values have to be these values otherwise the gazebo camera image
         won't be aligned properly with the frame it is supposedly originating from -->
-    <xacro:sensor_d435 parent="${prefix}base_link">
+    <xacro:sensor_d435 parent="${prefix}base_link" tf_prefix="${prefix}">
       <origin xyz="0.42 0 0.27" rpy="0 0.2 0"/>
     </xacro:sensor_d435>

Commit message: Published topic names sound correct in rostopic list. BUT in rqt_graph the topics arent visible. They should be in the namespace.

File: MiR200-with-UR5/mir_ur5_description/urdf/include/_d435.urdf.xacro (robot description, xacro)
@@ -9,5 +9,5 @@
   <!--File includes-->
   <xacro:include filename="$(find mir_ur5_description)/urdf/include/_d435.gazebo.xacro"/>
-  <xacro:macro name="sensor_d435" params="name:=camera topics_ns:=camera parent tf_prefix *origin">
+  <xacro:macro name="sensor_d435" params="name:=/camera topics_ns parent tf_prefix *origin">
     <xacro:property name="M_PI" value="3.1415926535897931" />
     <!-- The following values are approximate, and the camera node
@@ -119,5 +119,5 @@
     <link name="${tf_prefix}${name}_color_optical_frame"/>
     <!-- Realsense Gazebo Plugin -->
-    <xacro:gazebo_d435 camera_name="${name}" reference_link="${tf_prefix}${name}_link" topics_ns="${topics_ns}" depth_optical_frame="${tf_prefix}${name}_depth_optical_frame" color_optical_frame="${tf_prefix}${name}_color_optical_frame" infrared1_optical_frame="${tf_prefix}${name}_left_ir_optical_frame" infrared2_optical_frame="${tf_prefix}${name}_right_ir_optical_frame"/>
+    <xacro:gazebo_d435 camera_name="${name}" reference_link="${tf_prefix}${name}_link" topics_ns="${topics_ns}${name}" depth_optical_frame="${tf_prefix}${name}_depth_optical_frame" color_optical_frame="${tf_prefix}${name}_color_optical_frame" infrared1_optical_frame="${tf_prefix}${name}_left_ir_optical_frame" infrared2_optical_frame="${tf_prefix}${name}_right_ir_optical_frame"/>
   </xacro:macro>
 </robot>

File: MiR200-with-UR5/mir_ur5_description/urdf/mir_200_v1.urdf.xacro (robot description, xacro)
@@ -130,5 +130,5 @@
     </gazebo>
   </xacro:macro>
-  <xacro:macro name="mir_200" params="prefix">
+  <xacro:macro name="mir_200" params="ns_prefix prefix">
     <link name="${prefix}base_footprint" />
     <joint name="${prefix}base_joint" type="fixed">
@@ -257,5 +257,5 @@
     <!-- these values have to be these values otherwise the gazebo camera image
         won't be aligned properly with the frame it is supposedly originating from -->
-    <xacro:sensor_d435 parent="${prefix}base_link" tf_prefix="${prefix}">
+    <xacro:sensor_d435 parent="${prefix}base_link" topics_ns="${ns_prefix}" tf_prefix="${prefix}">
       <origin xyz="0.42 0 0.27" rpy="0 0.2 0"/>
     </xacro:sensor_d435>

File: MiR200-with-UR5/mir_ur5_description/urdf/mir_ur5.urdf.xacro (robot description, xacro)
@@ -17,5 +17,5 @@
         <xacro:arg name="tf_prefix" value="$(arg tf_prefix)"/>
     </xacro:include>
-    <xacro:mir_200 prefix="$(arg tf_prefix)"/>
+    <xacro:mir_200 ns_prefix="$(arg robot_namespace)" prefix="$(arg tf_prefix)"/>
     <!--The position of the model was measured using laser scachild_frame="$(arg tf_prefix)wrist_3_link_ur5" nner. See Florian's master thesis-->
     <joint name="robot_to_ur5" type="fixed">

Commit message: Attached D435 Plugin to MiR_Base and Ur5_Arm. Published Topics and tf_tree seems to be correct. Only the camera_Mount is missing.

File: MiR200-with-UR5/mir_ur5_description/urdf/include/_d435.urdf.xacro (robot description, xacro)
@@ -9,5 +9,5 @@
   <!--File includes-->
   <xacro:include filename="$(find mir_ur5_description)/urdf/include/_d435.gazebo.xacro"/>
-  <xacro:macro name="sensor_d435" params="name:=/camera topics_ns parent tf_prefix *origin">
+  <xacro:macro name="sensor_d435" params="name topics_ns parent tf_prefix *origin">
     <xacro:property name="M_PI" value="3.1415926535897931" />
     <!-- The following values are approximate, and the camera node

File: MiR200-with-UR5/mir_ur5_description/urdf/mir_200_v1.urdf.xacro (robot description, xacro)
@@ -257,5 +257,5 @@
     <!-- these values have to be these values otherwise the gazebo camera image
         won't be aligned properly with the frame it is supposedly originating from -->
-    <xacro:sensor_d435 parent="${prefix}base_link" topics_ns="${ns_prefix}" tf_prefix="${prefix}">
+    <xacro:sensor_d435 name="/camera_base" parent="${prefix}base_link" topics_ns="${ns_prefix}" tf_prefix="${prefix}">
       <origin xyz="0.42 0 0.27" rpy="0 0.2 0"/>
     </xacro:sensor_d435>

File: MiR200-with-UR5/mir_ur5_description/urdf/mir_ur5.urdf.xacro (robot description, xacro)
@@ -13,7 +13,7 @@
     <!--Include all needed urdf files-->
     <xacro:include filename="$(find mir_ur5_description)/urdf/mir_200_v1.urdf.xacro"/>
-    <!-- <xacro:include filename="$(find mir_ur5_description)/urdf/ur5.urdf.xacro"/> -->
     <xacro:include filename="$(find mir_ur5_description)/urdf/ur5_robot.urdf.xacro">
         <xacro:arg name="tf_prefix" value="$(arg tf_prefix)"/>
+        <xacro:arg name="robot_namespace" value="$(arg robot_namespace)"/>
     </xacro:include>
     <xacro:mir_200 ns_prefix="$(arg robot_namespace)" prefix="$(arg tf_prefix)"/>

File: MiR200-with-UR5/mir_ur5_description/urdf/ur5.urdf.xacro (robot description, xacro)
@@ -5,4 +5,5 @@
   <xacro:include filename="$(find mir_ur5_description)/urdf/include/ur.transmission_switch.xacro" />
   <xacro:include filename="$(find mir_ur5_description)/urdf/ur.gazebo.xacro" />
+  <xacro:include filename="$(find mir_ur5_description)/urdf/include/_d435.urdf.xacro"/>
   <xacro:macro name="cylinder_inertial" params="radius length mass *origin">
     <inertial>
@@ -14,5 +15,5 @@
     </inertial>
   </xacro:macro>
-  <xacro:macro name="ur5_robot" params="prefix joint_limited
+  <xacro:macro name="ur5_robot" params="prefix ns_prefix joint_limited
     shoulder_pan_lower_limit:=${-pi}    shoulder_pan_upper_limit:=${pi}
     shoulder_lift_lower_limit:=${-pi}    shoulder_lift_upper_limit:=${pi}
@@ -290,5 +291,5 @@
     </gazebo>
     <!-- optional: Attach a compliance tool link -->
-    <!-- <joint name="${prefix}tool_joint_ur5" type="fixed">
+    <joint name="${prefix}tool_joint_ur5" type="fixed">
       <origin xyz="0 ${wrist_3_length /2.0} 0" rpy="${-pi / 2.0} 0 ${pi / 2.0}"/>
       <parent link="${prefix}wrist_3_link_ur5"/>
@@ -304,6 +305,5 @@
         </visual>
     </link>
-  -->
-  <!--  <gazebo reference="${prefix}tool_link_ur5">
+  <gazebo reference="${prefix}tool_link_ur5">
       <kp value="0.0"/>
       <kd value="1.0"/>
@@ -311,5 +311,4 @@
       <maxVel value="0"/>
     </gazebo>
-  -->
     <joint name="${prefix}ee_fixed_joint" type="fixed">
       <origin xyz="${wrist_3_length/2.0} 0.0 0.0" rpy="0.0 ${pi/2.0} 0.0" /> <!-- rpy="0.0 0.0 ${pi/2.0}" -->
@@ -354,4 +353,7 @@
       <child link="${prefix}tool0"/>
     </joint> -->
+    <xacro:sensor_d435 name="/camera_arm" parent="${prefix}tool_link_ur5" topics_ns="${ns_prefix}" tf_prefix="${prefix}">
+      <origin xyz="${wrist_3_length/2.0} 0 0" rpy="-${pi/2.0} 0 0"/>
+    </xacro:sensor_d435>
   </xacro:macro>
 </robot>

File: MiR200-with-UR5/mir_ur5_description/urdf/ur5_robot.urdf.xacro (robot description, xacro)
@@ -7,4 +7,5 @@
   <xacro:arg name="transmission_hw_interface2" default="hardware_interface/VelocityJointInterface"/>
   <xacro:arg name="tf_prefix" default=''/>
+  <xacro:arg name="robot_namespace" default=''/>
   <!-- common stuff -->
   <!-- <xacro:include filename="$(find ur_description)/urdf/common.gazebo.xacro" /> -->
@@ -12,5 +13,5 @@
   <xacro:include filename="$(find mir_ur5_description)/urdf/ur5.urdf.xacro" />
   <!-- arm -->
-  <xacro:ur5_robot prefix="$(arg tf_prefix)" joint_limited="true" transmission_hw_interface1="$(arg transmission_hw_interface1)" transmission_hw_interface2="$(arg transmission_hw_interface2)"/>
+  <xacro:ur5_robot prefix="$(arg tf_prefix)" ns_prefix="$(arg robot_namespace)" joint_limited="true" transmission_hw_interface1="$(arg transmission_hw_interface1)" transmission_hw_interface2="$(arg transmission_hw_interface2)"/>
   <!--As MoveIt! seems to have difficulties with finding plans for the UR with full joint limits [-2pi, 2pi],
   there is a joint_limited version using joint limits restricted to [-pi,pi]. In order to use this joint limited version set joint_limited="true"-->
